File: MCU.sch (KiCad schematic (older format))
At the start: 28 parts, among them J5 GPIO, SW1 RST, SW2 Boot, U3 RP2040, U4 W25Q128JVS, Y1 ABLS-12.000MHZ-B4-T

Commit message: Add pull up for i2c and change layout
Parts:
- U3: symbol MCU_RaspberryPi_RP2040:RP2040 -> DCF77_Horloge-rescue:RP2040-MCU_RaspberryPi_RP2040
Connections:
- net +3V3: now also J5.10 (Pin_10)
- net GND: now also J5.1 (Pin_1)
- net STATUS_BAT: now also U3.37 (GPIO25); no longer U3.2 (GPIO0)
- net GPIO15: no longer names the net of U3.18 (GPIO15)
- net GPIO15: no longer J5.1 (Pin_1)
- net GPIO23: no longer names the net of U3.35 (GPIO23)
- net GPIO23: no longer J5.9 (Pin_9)
- net GPIO24: no longer names the net of U3.36 (GPIO24)
- net GPIO24: no longer J5.10 (Pin_10)
- new net +5V: J5.9 (Pin_9)
Changed lines of the file:
@@
 $EndDescr
 $Comp
-L MCU_RaspberryPi_RP2040:RP2040 U3
+L DCF77_Horloge-rescue:RP2040-MCU_RaspberryPi_RP2040 U3
 U 1 1 61172778
 P 3750 4250
@@
 	2300 5050 2500 5050
 Connection ~ 2300 5050
-Text GLabel 5000 2950 2    50   Input ~ 0
+Text GLabel 5000 5450 2    50   Input ~ 0
 STATUS_BAT
 Text GLabel 5000 5650 2    50   Input ~ 0
@@
 $EndComp
 Wire Wire Line
-	8250 4700 8750 4700
-Wire Wire Line
 	8250 4800 8750 4800
 Wire Wire Line
@@
 Wire Wire Line
 	8250 5400 8750 5400
-Wire Wire Line
-	8250 5500 8750 5500
-Wire Wire Line
-	8250 5600 8750 5600
-Text Label 8750 4700 2    50   ~ 0
-GPIO15
 Text Label 8750 4800 2    50   ~ 0
 GPIO16
@@
 Text Label 8750 5400 2    50   ~ 0
 GPIO22
-Text Label 8750 5500 2    50   ~ 0
-GPIO23
-Text Label 8750 5600 2    50   ~ 0
-GPIO24
-Wire Wire Line
-	5000 4450 5500 4450
 Wire Wire Line
 	5000 4550 5500 4550
@@
 Wire Wire Line
 	5000 5150 5500 5150
-Wire Wire Line
-	5000 5250 5500 5250
-Wire Wire Line
-	5000 5350 5500 5350
-Text Label 5500 4450 2    50   ~ 0
-GPIO15
 Text Label 5500 4550 2    50   ~ 0
 GPIO16
@@
 Text Label 5500 5150 2    50   ~ 0
 GPIO22
-Text Label 5500 5250 2    50   ~ 0
-GPIO23
-Text Label 5500 5350 2    50   ~ 0
-GPIO24
 Text Label 9850 3200 2    50   ~ 0
 QSPI_SD3
+$Comp
+L power:GND #PWR0101
+U 1 1 6120ED65
+P 8250 4700
+F 0 "#PWR0101" H 8250 4450 50  0001 C CNN
+F 1 "GND" H 8255 4527 50  0000 C CNN
+F 2 "" H 8250 4700 50  0001 C CNN
+F 3 "" H 8250 4700 50  0001 C CNN
+	1    8250 4700
+	0    -1   -1   0
+$EndComp
+$Comp
+L power:+3.3V #PWR0102
+U 1 1 6122B9EF
+P 8750 5600
+F 0 "#PWR0102" H 8750 5450 50  0001 C CNN
+F 1 "+3.3V" V 8750 5850 50  0000 C CNN
+F 2 "" H 8750 5600 50  0001 C CNN
+F 3 "" H 8750 5600 50  0001 C CNN
+	1    8750 5600
+	0    1    1    0
+$EndComp
+Wire Wire Line
+	8250 5600 8750 5600
+$Comp
+L power:+5V #PWR0103
+U 1 1 612300E3
+P 8750 5500
+F 0 "#PWR0103" H 8750 5350 50  0001 C CNN
+F 1 "+5V" V 8750 5600 50  0000 L CNN
+F 2 "" H 8750 5500 50  0001 C CNN
+F 3 "" H 8750 5500 50  0001 C CNN
+	1    8750 5500
+	0    1    1    0
+$EndComp
+Wire Wire Line
+	8250 5500 8750 5500
 $EndSCHEMATC

Commit message: change MCU from RP2040 to ESP32-WROOM-32
Parts:
- U3: symbol DCF77_Horloge-rescue:RP2040-MCU_RaspberryPi_RP2040 -> DCF77_Horloge-rescue:RP2040-MCU_RaspberryPi_RP2040-DCF77_Horloge-rescue
Changed lines of the file:
@@
 $EndDescr
 $Comp
-L DCF77_Horloge-rescue:RP2040-MCU_RaspberryPi_RP2040 U3
+L DCF77_Horloge-rescue:RP2040-MCU_RaspberryPi_RP2040-DCF77_Horloge-rescue U3
 U 1 1 61172778
 P 3750 4250
+AR Path="/61172778" Ref="U3"  Part="1"
+AR Path="/61171C55/61172778" Ref="U3"  Part="1"
 F 0 "U3" H 2500 6100 50  0000 C CNN
 F 1 "RP2040" H 4500 2300 50  0000 C CNN
