File: DCF77_Horloge.sch (KiCad schematic (older format))
At the start: 29 parts, among them J3 Conn_Display, Q1 AO3401A, U1 MCP73831-2-OT, U2 NCP1117-3.3_SOT223

Commit message: some changes
Parts:
- added C10: 0.1uF, Capacitor_SMD:C_0603_1608Metric_Pad1.08x0.95mm_HandSolder, symbol Device:C
- added R4: 560, Resistor_SMD:R_0603_1608Metric_Pad0.98x0.95mm_HandSolder, symbol Device:R
- added R5: 10k, Resistor_SMD:R_0603_1608Metric_Pad0.98x0.95mm_HandSolder, symbol Device:R
- added SW1: RST, Button_Switch_SMD:SW_SPST_FSMSM, symbol Switch:SW_Push
- J1: renamed from J?; footprint (none) -> Connector_USB:USB_C_Receptacle_GCT_USB4085; symbol Connector:USB_C_Receptacle_USB2.0 -> DCF77_Horloge-rescue:USB_C_Receptacle_USB2.0-Connector
- SW2: renamed from SW?; footprint (none) -> Button_Switch_SMD:SW_SPST_FSMSM
- gave numbers to parts that had none: 7
Connections:
- net +3V3: now also R5.2
- net BOOT: now also C10.2, R5.1
- net GND: now also C6.1, C10.1, SW1.2; no longer C6.2
- net RST: now also R4.2; no longer C6.1
- net SCL: now also U3.33 (IO39)
- net SDA: now also U3.36 (IO42)
- new net: C6.2, R4.1, SW1.1
Other:
- moved on the sheet: C6, C9, R3
Changed lines of the file:
@@
 	10400 1000 10500 1000
 $Comp
-L Connector:USB_C_Receptacle_USB2.0 J?
+L DCF77_Horloge-rescue:USB_C_Receptacle_USB2.0-Connector J1
 U 1 1 615020ED
 P 1850 1650
-F 0 "J?" H 1957 2517 50  0000 C CNN
+F 0 "J1" H 1957 2517 50  0000 C CNN
 F 1 "USB_C_Receptacle_USB2.0" H 1957 2426 50  0000 C CNN
-F 2 "" H 2000 1650 50  0001 C CNN
+F 2 "Connector_USB:USB_C_Receptacle_GCT_USB4085" H 2000 1650 50  0001 C CNN
 F 3 "https://www.usb.org/sites/default/files/documents/usb_type-c.zip" H 2000 1650 50  0001 C CNN
 	1    1850 1650
@@
 NoConn ~ 2450 2250
 $Comp
-L Device:C C?
+L Device:C C8
 U 1 1 61628ECF
 P 1700 3550
-F 0 "C?" H 1750 3450 50  0000 C CNN
+F 0 "C8" H 1750 3450 50  0000 C CNN
 F 1 "10uF" H 1800 3650 50  0000 C CNN
 F 2 "Capacitor_SMD:C_0603_1608Metric_Pad1.08x0.95mm_HandSolder" H 1738 3400 50  0001 C CNN
@@
 $EndComp
 $Comp
-L Device:C C?
+L Device:C C9
 U 1 1 6162D311
-P 2000 3550
-F 0 "C?" H 1950 3450 50  0000 C CNN
-F 1 "0.1uF" H 1900 3650 50  0000 C CNN
-F 2 "Capacitor_SMD:C_0603_1608Metric_Pad1.08x0.95mm_HandSolder" H 2038 3400 50  0001 C CNN
-F 3 "~" H 2000 3550 50  0001 C CNN
-	1    2000 3550
+P 2050 3550
+F 0 "C9" H 2000 3450 50  0000 C CNN
+F 1 "0.1uF" H 1950 3650 50  0000 C CNN
+F 2 "Capacitor_SMD:C_0603_1608Metric_Pad1.08x0.95mm_HandSolder" H 2088 3400 50  0001 C CNN
+F 3 "~" H 2050 3550 50  0001 C CNN
+	1    2050 3550
 	-1   0    0    1
 $EndComp
@@
 	1700 3700 1850 3700
 $Comp
-L power:+3.3V #PWR?
+L power:+3.3V #PWR016
 U 1 1 61636269
 P 1850 3400
-F 0 "#PWR?" H 1850 3250 50  0001 C CNN
+F 0 "#PWR016" H 1850 3250 50  0001 C CNN
 F 1 "+3.3V" H 1865 3573 50  0000 C CNN
 F 2 "" H 1850 3400 50  0001 C CNN
@@
 Connection ~ 1850 3400
 Wire Wire Line
-	1850 3400 2000 3400
-$Comp
-L power:GND #PWR?
+	1850 3400 2050 3400
+$Comp
+L power:GND #PWR019
 U 1 1 616380DA
 P 1850 3700
-F 0 "#PWR?" H 1850 3450 50  0001 C CNN
+F 0 "#PWR019" H 1850 3450 50  0001 C CNN
 F 1 "GND" H 1855 3527 50  0000 C CNN
 F 2 "" H 1850 3700 50  0001 C CNN
@@
 $EndComp
 Connection ~ 1850 3700
-Wire Wire Line
-	1850 3700 1950 3700
-Connection ~ 2000 3400
-$Comp
-L Device:C C?
+Connection ~ 2050 3400
+$Comp
+L Device:C C6
 U 1 1 6163D1DD
-P 2300 3800
-F 0 "C?" H 2250 3700 50  0000 C CNN
-F 1 "0.1uF" H 2200 3900 50  0000 C CNN
-F 2 "Capacitor_SMD:C_0603_1608Metric_Pad1.08x0.95mm_HandSolder" H 2338 3650 50  0001 C CNN
-F 3 "~" H 2300 3800 50  0001 C CNN
-	1    2300 3800
-	0    1    1    0
-$EndComp
-$Comp
-L Device:R R?
+P 900 4750
+F 0 "C6" H 850 4650 50  0000 C CNN
+F 1 "0.1uF" H 800 4850 50  0000 C CNN
+F 2 "Capacitor_SMD:C_0603_1608Metric_Pad1.08x0.95mm_HandSolder" H 938 4600 50  0001 C CNN
+F 3 "~" H 900 4750 50  0001 C CNN
+	1    900  4750
+	-1   0    0    1
+$EndComp
+$Comp
+L Device:R R3
 U 1 1 6163DF8F
-P 2700 3600
-F 0 "R?" H 2850 3550 50  0000 R CNN
-F 1 "10k" H 2850 3650 50  0000 R CNN
-F 2 "Resistor_SMD:R_0603_1608Metric_Pad0.98x0.95mm_HandSolder" V 2630 3600 50  0001 C CNN
-F 3 "~" H 2700 3600 50  0001 C CNN
-	1    2700 3600
-	-1   0    0    1
-$EndComp
-Wire Wire Line
-	2000 3400 2700 3400
+P 1300 4000
+F 0 "R3" V 1400 4050 50  0000 R CNN
+F 1 "10k" V 1300 4100 50  0000 R CNN
+F 2 "Resistor_SMD:R_0603_1608Metric_Pad0.98x0.95mm_HandSolder" V 1230 4000 50  0001 C CNN
+F 3 "~" H 1300 4000 50  0001 C CNN
+	1    1300 4000
+	-1   0    0    1
+$EndComp
+Wire Wire Line
+	2050 3400 2700 3400
 Wire Wire Line
 	2700 3400 2700 3450
 Connection ~ 2700 3400
 Wire Wire Line
-	2700 3750 2700 3800
-Wire Wire Line
-	2450 3800 2700 3800
-Connection ~ 2700 3800
-Wire Wire Line
-	1950 3700 1950 3800
-Wire Wire Line
-	1950 3800 2150 3800
-Connection ~ 1950 3700
-Wire Wire Line
-	1950 3700 2000 3700
-$Comp
-L Switch:SW_Push SW?
+	1300 4150 1300 4200
+$Comp
+L Switch:SW_Push SW2
 U 1 1 6167B561
 P 2200 4350
-F 0 "SW?" H 2200 4550 50  0000 C CNN
+F 0 "SW2" H 2200 4550 50  0000 C CNN
 F 1 "boot" H 2200 4500 50  0000 C CNN
-F 2 "" H 2200 4550 50  0001 C CNN
+F 2 "Button_Switch_SMD:SW_SPST_FSMSM" H 2200 4550 50  0001 C CNN
 F 3 "~" H 2200 4550 50  0001 C CNN
 	1    2200 4350
@@
 $EndComp
 $Comp
-L power:GND #PWR?
+L power:GND #PWR015
 U 1 1 6167D27E
 P 1800 4350
-F 0 "#PWR?" H 1800 4100 50  0001 C CNN
+F 0 "#PWR015" H 1800 4100 50  0001 C CNN
 F 1 "GND" H 1805 4177 50  0000 C CNN
 F 2 "" H 1800 4350 50  0001 C CNN
@@
 $EndComp
 Wire Wire Line
-	2950 4350 2400 4350
+	2950 4350 2750 4350
 Wire Wire Line
 	2000 4350 1800 4350
 Text Label 2700 4350 2    50   ~ 0
 BOOT
-Text Label 2550 3800 0    50   ~ 0
+Text Label 1350 4200 0    50   ~ 0
 RST
 $Comp
-L RF_Module:ESP32-S2-WROVER U?
+L RF_Module:ESP32-S2-WROVER U3
 U 1 1 616E884A
 P 3550 5250
-F 0 "U?" H 3100 6400 50  0000 C CNN
+F 0 "U3" H 3100 6400 50  0000 C CNN
 F 1 "ESP32-S2-WROVER" H 3100 4200 50  0000 C CNN
 F 2 "RF_Module:ESP32-S2-WROVER" H 4300 4100 50  0001 C CNN
@@
 $EndComp
 Wire Wire Line
-	2950 3800 2950 4250
-Wire Wire Line
-	2700 3800 2950 3800
+	2950 3850 2950 4250
 Wire Wire Line
 	3550 3400 3550 4050
@@
 	2700 3400 3550 3400
 $Comp
-L power:GND #PWR?
+L power:GND #PWR021
 U 1 1 6176AE30
 P 3550 6350
-F 0 "#PWR?" H 3550 6100 50  0001 C CNN
+F 0 "#PWR021" H 3550 6100 50  0001 C CNN
 F 1 "GND" H 3555 6177 50  0000 C CNN
 F 2 "" H 3550 6350 50  0001 C CNN
@@
 $EndComp
 $Comp
-L Device:R R?
+L Device:R R6
 U 1 1 617B0682
 P 2950 2050
-F 0 "R?" H 3100 2050 50  0000 R CNN
+F 0 "R6" H 3100 2050 50  0000 R CNN
 F 1 "5k1" V 2950 2150 50  0000 R CNN
 F 2 "Resistor_SMD:R_0603_1608Metric_Pad0.98x0.95mm_HandSolder" V 2880 2050 50  0001 C CNN
@@
 $EndComp
 $Comp
-L Device:R R?
+L Device:R R7
 U 1 1 617B2832
 P 3150 2050
-F 0 "R?" H 3300 2050 50  0000 R CNN
+F 0 "R7" H 3300 2050 50  0000 R CNN
 F 1 "5k1" V 3150 2150 50  0000 R CNN
 F 2 "Resistor_SMD:R_0603_1608Metric_Pad0.98x0.95mm_HandSolder" V 3080 2050 50  0001 C CNN
@@
 Wire Wire Line
 	4400 5950 4150 5950
+$Comp
+L Device:R R5
+U 1 1 618ED136
+P 2750 4200
+F 0 "R5" H 2900 4150 50  0000 R CNN
+F 1 "10k" V 2750 4300 50  0000 R CNN
+F 2 "Resistor_SMD:R_0603_1608Metric_Pad0.98x0.95mm_HandSolder" V 2680 4200 50  0001 C CNN
+F 3 "~" H 2750 4200 50  0001 C CNN
+	1    2750 4200
+	-1   0    0    1
+$EndComp
+Connection ~ 2750 4350
+Wire Wire Line
+	2750 4350 2400 4350
+$Comp
+L power:+3.3V #PWR020
+U 1 1 618ED63F
+P 2750 4050
+F 0 "#PWR020" H 2750 3900 50  0001 C CNN
+F 1 "+3.3V" H 2750 4200 50  0000 C CNN
+F 2 "" H 2750 4050 50  0001 C CNN
+F 3 "" H 2750 4050 50  0001 C CNN
+	1    2750 4050
+	1    0    0    -1
+$EndComp
+Wire Wire Line
+	1850 3700 2050 3700
+Wire Wire Line
+	2050 3850 2050 4200
+Wire Wire Line
+	2050 4200 1300 4200
+Wire Wire Line
+	2050 3850 2950 3850
+$Comp
+L Device:R R4
+U 1 1 619053C7
+P 1300 4350
+F 0 "R4" V 1400 4400 50  0000 R CNN
+F 1 "560" V 1300 4450 50  0000 R CNN
+F 2 "Resistor_SMD:R_0603_1608Metric_Pad0.98x0.95mm_HandSolder" V 1230 4350 50  0001 C CNN
+F 3 "~" H 1300 4350 50  0001 C CNN
+	1    1300 4350
+	-1   0    0    1
+$EndComp
+Connection ~ 1300 4200
+$Comp
+L Switch:SW_Push SW1
+U 1 1 6190579D
+P 1300 4750
+F 0 "SW1" H 1300 4950 50  0000 C CNN
+F 1 "RST" H 1300 4900 50  0000 C CNN
+F 2 "Button_Switch_SMD:SW_SPST_FSMSM" H 1300 4950 50  0001 C CNN
+F 3 "~" H 1300 4950 50  0001 C CNN
+	1    1300 4750
+	0    1    1    0
+$EndComp
+Wire Wire Line
+	1300 4500 1300 4550
+Wire Wire Line
+	1300 4550 900  4550
+Wire Wire Line
+	900  4550 900  4600
+Connection ~ 1300 4550
+Wire Wire Line
+	900  4900 900  5050
+Wire Wire Line
+	900  5050 1100 5050
+Wire Wire Line
+	1300 5050 1300 4950
+$Comp
+L power:GND #PWR010
+U 1 1 6190EF23
+P 1100 5050
+F 0 "#PWR010" H 1100 4800 50  0001 C CNN
+F 1 "GND" H 1105 4877 50  0000 C CNN
+F 2 "" H 1100 5050 50  0001 C CNN
+F 3 "" H 1100 5050 50  0001 C CNN
+	1    1100 5050
+	1    0    0    -1
+$EndComp
+Connection ~ 1100 5050
+Wire Wire Line
+	1100 5050 1300 5050
+$Comp
+L power:+3.3V #PWR014
+U 1 1 61911F53
+P 1300 3850
+F 0 "#PWR014" H 1300 3700 50  0001 C CNN
+F 1 "+3.3V" H 1315 4023 50  0000 C CNN
+F 2 "" H 1300 3850 50  0001 C CNN
+F 3 "" H 1300 3850 50  0001 C CNN
+	1    1300 3850
+	1    0    0    -1
+$EndComp
+$Comp
+L Device:C C10
+U 1 1 6191275E
+P 2200 4550
+F 0 "C10" H 2150 4450 50  0000 C CNN
+F 1 "0.1uF" H 2100 4650 50  0000 C CNN
+F 2 "Capacitor_SMD:C_0603_1608Metric_Pad1.08x0.95mm_HandSolder" H 2238 4400 50  0001 C CNN
+F 3 "~" H 2200 4550 50  0001 C CNN
+	1    2200 4550
+	0    -1   -1   0
+$EndComp
+Wire Wire Line
+	2400 4350 2400 4550
+Wire Wire Line
+	2400 4550 2350 4550
+Connection ~ 2400 4350
+Wire Wire Line
+	2000 4350 2000 4550
+Wire Wire Line
+	2000 4550 2050 4550
+Connection ~ 2000 4350
+Wire Wire Line
+	4150 4950 4350 4950
+Wire Wire Line
+	4150 4650 4350 4650
+Text GLabel 4350 4950 2    50   Input ~ 0
+SCL
+Text GLabel 4350 4650 2    50   Input ~ 0
+SDA
 $EndSCHEMATC
