File: Screen.kicad_sch (KiCad schematic)
At the start: 17 parts, among them J2 FH34SRJ 24S, Q2 SK3424

Commit message: update
Parts:
- J2: footprint (none) -> AREA_lib_Connector:HRS_FH34SRJ-24S-0.5SH(99)
- Q2: symbol Simulation_SPICE:NMOS -> Device:Q_NMOS_GSD
Connections:
- net GDR: now also Q2.1 (G); no longer Q2.2 (G)
- net RESET: now also Q2.3 (D); no longer Q2.1 (D)
- net at C28.2, D5.2 (A), L2.2: now also Q2.2 (S); no longer Q2.3 (S)
Changed lines of the file:
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@@
     )
   )
-  (symbol (lib_id "Simulation_SPICE:NMOS") (at 163.83 41.91 180) (unit 1)
+  (symbol (lib_id "Device:Q_NMOS_GSD") (at 163.83 41.91 180) (unit 1)
     (in_bom yes) (on_board yes) (dnp no) (fields_autoplaced)
     (property "Reference" "Q2" (at 158.6231 41.2663 0)
@@
       (effects (font (size 1.27 1.27)) hide)
     )
-    (property "Datasheet" "https://ngspice.sourceforge.io/docs/ngspice-manual.pdf" (at 163.83 29.21 0)
+    (property "Datasheet" "~" (at 163.83 41.91 0)
       (effects (font (size 1.27 1.27)) hide)
     )
@@
       (effects (font (size 1.27 1.27)) (justify left))
     )
-    (property "Footprint" "" (at 190.5 71.12 0)
-      (effects (font (size 1.27 1.27)) hide)
-    )
+    (property "Footprint" "AREA_lib_Connector:HRS_FH34SRJ-24S-0.5SH(99)" (at 190.5 71.12 0)
+      (effects (font (size 1.27 1.27)) hide)
+    )
