File: DCF77_Horloge.kicad_pcb (KiCad board)
At the start: 2 copper layers, 98.6 x 61.3 mm, 33 parts, among them J1 USB_C_Receptacle_USB2.0, J3 Conn_Display, Q1 AO3401A, SW1 RST, SW2 boot, U1 MCP73831-2-OT, U2 NCP1117-3.3_SOT223, U3 ESP32-S2-WROVER

Commit message: big update
Parts:
- removed R9: 2K, Resistor_SMD:R_0603_1608Metric_Pad1.05x0.95mm_HandSolder
- removed SW2: boot, Button_Switch_SMD:SW_SPST_FSMSM
- added C11: 100n, Capacitor_SMD:C_0603_1608Metric, F.Cu at (225.5, 63.3)
- added C12: 100n, Capacitor_SMD:C_0603_1608Metric, F.Cu at (225.5, 65.8)
- added C13: 10u, Capacitor_SMD:C_0603_1608Metric, F.Cu at (225.5, 68.3)
- added C14: 100n, Capacitor_SMD:C_0603_1608Metric, F.Cu at (225.5, 70.8)
- added C15: 4.7u, Capacitor_SMD:C_0603_1608Metric, F.Cu at (144.2, 61.0)
- added C16: 22u, Capacitor_SMD:C_0805_2012Metric, F.Cu at (144.5, 64.2)
- added C17: 22u, Capacitor_SMD:C_0805_2012Metric, F.Cu at (146.5, 64.2)
- added C18: 100n, Capacitor_SMD:C_0603_1608Metric, F.Cu at (171.0, 75.0)
- added C19: 100n, Capacitor_SMD:C_0603_1608Metric, F.Cu at (150.5, 59.0)
- added C20: 100n, Capacitor_SMD:C_0603_1608Metric, F.Cu at (164.7, 55.7)
- added C21: 1u/25V, Capacitor_SMD:C_0603_1608Metric, F.Cu at (213.7, 63.3)
- added C22: 4.7u, Capacitor_SMD:C_0603_1608Metric, F.Cu at (166.2, 55.7)
- added C23: 1u/25V, Capacitor_SMD:C_0603_1608Metric, F.Cu at (213.7, 65.8)
- added C24: 1u/25V, Capacitor_SMD:C_0603_1608Metric, F.Cu at (213.7, 68.3)
- added C25: 1u/25V, Capacitor_SMD:C_0603_1608Metric, F.Cu at (213.7, 70.8)
- added C26: 1u/25V, Capacitor_SMD:C_0603_1608Metric, F.Cu at (213.7, 73.3)
- added C27: 1u/25V, Capacitor_SMD:C_0603_1608Metric, F.Cu at (213.7, 75.8)
- added C28: 4.7u/25V, Capacitor_SMD:C_0603_1608Metric, F.Cu at (213.7, 78.3)
- added C29: 1u/25V, Capacitor_SMD:C_0603_1608Metric, F.Cu at (213.7, 80.8)
- added C30: 100n, Capacitor_SMD:C_0603_1608Metric, F.Cu at (213.7, 83.4)
- added D2: LED_DEBUG, LED_SMD:LED_0603_1608Metric, F.Cu at (242.8, 69.3)
- added D3: LED_5V, LED_SMD:LED_0603_1608Metric, F.Cu at (146.0, 66.8)
- added D4: SS2040, Diode_SMD:D_SOD-123, F.Cu at (138.0, 63.8)
- added D5: SS2040, Diode_SMD:D_SOD-123, F.Cu at (218.7, 63.7)
- added D6: SS2040, Diode_SMD:D_SOD-123, F.Cu at (218.7, 67.0)
- added D7: SS2040, Diode_SMD:D_SOD-123, F.Cu at (218.7, 70.4)
- added L1: DFE201612E-2R2M=P2, Inductor_SMD:L_0805_2012Metric_Pad1.15x1.40mm_HandSolder, F.Cu at (135.8, 61.2)
- added L2: L, Inductor_SMD:L_1210_3225Metric, F.Cu at (218.5, 74.2)
- added Q2: SK3424, Package_TO_SOT_SMD:SC-59, F.Cu at (218.2, 78.6)
- added R10: 4k7, Resistor_SMD:R_0603_1608Metric, F.Cu at (166.0, 71.5)
- added R11: 300m, Resistor_SMD:R_2512_6332Metric, F.Cu at (147.0, 57.2)
- added R12: 1.5k, Resistor_SMD:R_0603_1608Metric, F.Cu at (229.5, 73.3)
- added R13: 330, Resistor_SMD:R_0603_1608Metric, F.Cu at (143.1, 66.8)
- added R14: 4k7, Resistor_SMD:R_0603_1608Metric, F.Cu at (156.5, 56.9)
- added R15: 4k7, Resistor_SMD:R_0603_1608Metric, F.Cu at (156.5, 59.9)
- added R16: 0, Resistor_SMD:R_0603_1608Metric, F.Cu at (153.8, 55.2)
- added R17: 0, Resistor_SMD:R_0603_1608Metric, F.Cu at (153.8, 53.8)
- added R18: 2M, Resistor_SMD:R_0603_1608Metric, F.Cu at (158.2, 55.7)
- added R19: 4M, Resistor_SMD:R_0603_1608Metric, F.Cu at (159.7, 55.7)
- added SW3: RST, Button_Switch_SMD:SW_SPST_CK_RS282G05A3, F.Cu at (241.0, 78.0)
- added U4: TPS613222ADBV, Package_TO_SOT_SMD:SOT-23-5, F.Cu at (141.2, 63.2)
- added U5: HDC1080, Package_SON:Texas_PWSON-N6, F.Cu at (167.4, 74.9)
- added U6: INA219AxDCN, Package_TO_SOT_SMD:SOT-23-8, F.Cu at (153.2, 57.8)
- added U7: TLV8811DBV, Package_TO_SOT_SMD:SOT-23-5, F.Cu at (162.2, 55.2)
- added Y1: 8MHz, Crystal:Crystal_SMD_5032-4Pin_5.0x3.2mm, F.Cu at (226.9, 82.0)
- C1, C4, C5: footprint Capacitor_SMD:C_0603_1608Metric_Pad1.08x0.95mm_HandSolder -> Capacitor_SMD:C_0603_1608Metric
- C10, C9: value 0.1uF -> 100n; footprint Capacitor_SMD:C_0603_1608Metric_Pad1.08x0.95mm_HandSolder -> Capacitor_SMD:C_0603_1608Metric
- C2: footprint Capacitor_THT:CP_Radial_D5.0mm_P2.00mm -> Capacitor_SMD:CP_Elec_5x5.4
- C3: value 4.7uF -> 4.7u; footprint Capacitor_SMD:C_0603_1608Metric_Pad1.08x0.95mm_HandSolder -> Capacitor_SMD:C_0603_1608Metric
- C6: value 0.1uF -> 18p; footprint Capacitor_SMD:C_0603_1608Metric_Pad1.08x0.95mm_HandSolder -> Capacitor_SMD:C_0603_1608Metric
- C7: value 10u -> 1u/25V; footprint Capacitor_THT:CP_Radial_D5.0mm_P2.50mm -> Capacitor_SMD:C_0603_1608Metric
- C8: value 10uF -> 18p; footprint Capacitor_SMD:C_0603_1608Metric_Pad1.08x0.95mm_HandSolder -> Capacitor_SMD:C_0603_1608Metric
- D1: value B5819W SL -> SS2040
- J3: value Conn_Display -> Conn_01x04_Socket; footprint Connector_PinSocket_2.54mm:PinSocket_1x04_P2.54mm_Vertical -> Connector_PinHeader_2.54mm:PinHeader_1x04_P2.54mm_Vertical
- R1, R2, R6, R7: footprint Resistor_SMD:R_0603_1608Metric_Pad0.98x0.95mm_HandSolder -> Resistor_SMD:R_0603_1608Metric
- R3: value 10k -> 270; footprint Resistor_SMD:R_0603_1608Metric_Pad0.98x0.95mm_HandSolder -> Resistor_SMD:R_0603_1608Metric
- R4: value 560 -> 10k; footprint Resistor_SMD:R_0603_1608Metric_Pad0.98x0.95mm_HandSolder -> Resistor_SMD:R_0603_1608Metric
- R5: value 10k -> 4k7; footprint Resistor_SMD:R_0603_1608Metric_Pad0.98x0.95mm_HandSolder -> Resistor_SMD:R_0603_1608Metric
- R8: value 2K -> 0.47; footprint Resistor_SMD:R_0603_1608Metric_Pad1.05x0.95mm_HandSolder -> Resistor_SMD:R_0603_1608Metric
- SW1: value RST -> BOOT; footprint Button_Switch_SMD:SW_SPST_FSMSM -> Button_Switch_SMD:SW_SPST_CK_RS282G05A3
- U3: value ESP32-S2-WROVER -> STM32F302C6Tx; footprint RF_Module:ESP32-S2-WROVER -> Package_QFP:LQFP-48_7x7mm_P0.5mm
- moved R7 90.7 mm to (104.0, 63.8), turned to 0 degrees
- moved R6 89.1 mm to (104.1, 51.5), turned to 180 degrees
- moved J1 88.0 mm to (105.0, 60.7), turned to 90 degrees
- moved R5 46.1 mm to (168.8, 71.5)
- moved C2 34.7 mm to (130.5, 57.0)
- moved C1 34.4 mm to (107.0, 60.5), turned to -90 degrees
- moved C5 25.8 mm to (133.8, 70.2), turned to -90 degrees
- moved U2 25.4 mm to (128.5, 68.8), turned to 180 degrees
- moved R3 24.4 mm to (116.0, 81.2)
- moved C4 21.0 mm to (133.8, 67.2), turned to 90 degrees
- moved R2 18.3 mm to (130.5, 62.5)
- moved Q1 10.4 mm to (135.2, 55.1), turned to 0 degrees
- moved D1 9.88 mm to (138.2, 55.8), turned to 90 degrees
- moved U3 5.56 mm to (113.8, 70.2)
- moved U1 3.21 mm to (141.4, 55.2)
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Connections:
- net Net-(U3-Pad14) renamed /SPI_CS
- net Net-(U3-Pad18) renamed /DCF77_OUT
- net Net-(U3-Pad39) renamed /SPI_CLK
- C1 pad 1: +5V -> VBUS
- C10 pad 1: GND -> +3V3
- C10 pad 2: /BOOT -> GND
- C2 pad 1: +5V -> VBUS
- C4 pad 2: Net-(C4-Pad2) -> +5V
- C6 pad 1: GND -> Net-(U3-PF0)
- C6 pad 2: Net-(C6-Pad2) -> GND
- C7 pad 1: +3V3 -> GND
- C7 pad 2: GND -> Net-(J2-Pin_5)
- C8 pad 1: GND -> Net-(U3-PF1)
- C8 pad 2: +3V3 -> GND
- C9 pad 1: GND -> /RST
- C9 pad 2: +3V3 -> GND
- D1 pad 1: Net-(C4-Pad2) -> +5V
- D1 pad 2: +5V -> VBUS
- J1 pad A4: +5V -> VBUS
- J1 pad A6: USB+ -> /USB+
- J1 pad A7: USB- -> /USB-
- J1 pad A8: Net-(J1-PadA8) -> unconnected-(J1-SBU1-PadA8)
- J1 pad A9: +5V -> VBUS
- J1 pad B4: +5V -> VBUS
- J1 pad B6: USB+ -> /USB+
- J1 pad B7: USB- -> /USB-
- J1 pad B8: Net-(J1-PadB8) -> unconnected-(J1-SBU2-PadB8)
- J1 pad B9: +5V -> VBUS
- J3 pad 1: GND -> unconnected-(J3-Pin_1-Pad1)
- J3 pad 2: +3V3 -> unconnected-(J3-Pin_2-Pad2)
- J3 pad 3: SCL -> unconnected-(J3-Pin_3-Pad3)
- J3 pad 4: SDA -> unconnected-(J3-Pin_4-Pad4)
- Q1 pad 1: Net-(C4-Pad2) -> +5V
- Q1 pad 2: +5V -> VBUS
- Q1 pad 3: +BATT -> +5VD
- R2 pad 1: GND -> VBUS
- R2 pad 2: +5V -> GND
- R3 pad 1: /RST -> GND
- R3 pad 2: +3V3 -> Net-(D2-K)
- R4 pad 1: Net-(C6-Pad2) -> GND
- R4 pad 2: /RST -> /BOOT0
- R5 pad 1: /BOOT -> /SCL_HDC1080
- R8 pad 1: SCL -> /Screen/RESET
- R8 pad 2: +3V3 -> GND
- SW1 pad 1: Net-(C6-Pad2) -> +3V3
- SW1 pad 2: GND -> /BOOT0
- U1 pad 4: +5V -> VBUS
- U2 pad 3: Net-(C4-Pad2) -> +5V
- U3 pad 1: GND -> unconnected-(U3-VBAT-Pad1)
- U3 pad 10: Net-(U3-Pad10) -> /VBAT_SENSE
- U3 pad 11: Net-(U3-Pad11) -> unconnected-(U3-PA1-Pad11)
- U3 pad 12: Net-(U3-Pad12) -> unconnected-(U3-PA2-Pad12)
- U3 pad 13: Net-(U3-Pad13) -> unconnected-(U3-PA3-Pad13)
- U3 pad 15: Net-(U3-Pad15) -> unconnected-(U3-PA5-Pad15)
- U3 pad 16: Net-(U3-Pad16) -> unconnected-(U3-PA6-Pad16)
- U3 pad 17: Net-(U3-Pad17) -> unconnected-(U3-PA7-Pad17)
- U3 pad 19: Net-(U3-Pad19) -> unconnected-(U3-PB1-Pad19)
- U3 pad 2: +3V3 -> unconnected-(U3-PC13-Pad2)
- U3 pad 20: Net-(U3-Pad20) -> unconnected-(U3-PB2-Pad20)
- U3 pad 21: Net-(U3-Pad21) -> unconnected-(U3-PB10-Pad21)
- U3 pad 22: USB- -> unconnected-(U3-PB11-Pad22)
- U3 pad 23: USB+ -> GND
- U3 pad 24: Net-(U3-Pad24) -> +3V3
- U3 pad 25: Net-(U3-Pad25) -> unconnected-(U3-PB12-Pad25)
- U3 pad 26: GND -> unconnected-(U3-PB13-Pad26)
- U3 pad 27: Net-(U3-Pad27) -> unconnected-(U3-PB14-Pad27)
- U3 pad 28: Net-(U3-Pad28) -> unconnected-(U3-PB15-Pad28)
- U3 pad 29: Net-(U3-Pad29) -> unconnected-(U3-PA8-Pad29)
- U3 pad 3: /BOOT -> unconnected-(U3-PC14-Pad3)
- U3 pad 30: Net-(U3-Pad30) -> /SCL_INA219
- U3 pad 31: Net-(U3-Pad31) -> /SDA_INA219
- U3 pad 32: Net-(U3-Pad32) -> /USB-
- U3 pad 33: SCL -> /USB+
- U3 pad 34: Net-(U3-Pad34) -> unconnected-(U3-PA13-Pad34)
- U3 pad 35: Net-(U3-Pad35) -> GND
- U3 pad 36: SDA -> +3V3
- U3 pad 37: Net-(U3-Pad37) -> /SDA_HDC1080
- U3 pad 38: Net-(U3-Pad38) -> /SCL_HDC1080
- U3 pad 4: Net-(U3-Pad4) -> unconnected-(U3-PC15-Pad4)
- U3 pad 40: Net-(U3-Pad40) -> unconnected-(U3-PB4-Pad40)
- U3 pad 41: /RST -> /SPI_DATA
- U3 pad 42: GND -> /SCREEN_DC
- U3 pad 43: GND -> /SCREEN_RST_N
- U3 pad 5: Net-(U3-Pad5) -> Net-(U3-PF0)
- U3 pad 6: Net-(U3-Pad6) -> Net-(U3-PF1)
- U3 pad 7: Net-(U3-Pad7) -> /RST
- U3 pad 8: Net-(U3-Pad8) -> GND
- U3 pad 9: Net-(U3-Pad9) -> +3V3
Routing:
- net +5V: track 95.0 -> 0.00 mm
- net +3V3: track 82.3 -> 0.00 mm, vias 2 -> 0
- net SDA: track 78.3 -> 0.00 mm, vias 2 -> 0
- net SCL: track 72.6 -> 0.00 mm, vias 2 -> 0
- net USB-: track 69.9 -> 0.00 mm
- net USB+: track 69.9 -> 0.00 mm
- net /RST: track 52.7 -> 0.00 mm
- net +BATT: track 46.0 -> 0.00 mm
- net Net-(C4-Pad2): track 11.4 -> 0.00 mm
- net GND: track 7.45 -> 0.00 mm, vias 19 -> 0
- net Net-(J1-CC2): track 6.43 -> 0.00 mm
- net Net-(J1-CC1): track 6.06 -> 0.00 mm
- net Net-(C6-Pad2): track 4.36 -> 0.00 mm
- net Net-(U1-PROG): track 1.69 -> 0.00 mm
- removed copper zone on F.Cu, net +BATT
- removed copper zone on B.Cu, net GND
- removed copper zone on F.Cu, net GND
Other:
- net class Default removed

Commit message: update
Parts:
- added J2: FH34SRJ 24S, AREA_lib_Connector:HRS_FH34SRJ-24S-0.5SH(99), F.Cu at (195.5, 58.2)
- added Q3: SK3424, Package_TO_SOT_SMD:SC-59, F.Cu at (187.0, 54.0)
- added R9: 120, Resistor_SMD:R_0603_1608Metric, F.Cu at (184.2, 53.8)
- BT1: footprint Battery:BatteryHolder_MPD_BH-18650-PC2 -> Battery:BatteryHolder_Keystone_1042_1x18650
- J1: footprint Connector_USB:USB_C_Receptacle_GCT_USB4085 -> Connector_USB:USB_C_Receptacle_GCT_USB4105-xx-A_16P_TopMnt_Horizontal; moved to F.Cu
- J3: footprint Connector_PinHeader_2.54mm:PinHeader_1x04_P2.54mm_Vertical -> Connector_PinHeader_2.54mm:PinHeader_1x04_P2.54mm_Vertical_SMD_Pin1Left; moved to F.Cu
- R11: footprint Resistor_SMD:R_2512_6332Metric -> Resistor_SMD:R_0805_2012Metric
- moved D2 82.4 mm to (161.2, 57.2)
- moved SW3 76.0 mm to (165.1, 82.2)
- moved Y1 64.5 mm to (168.7, 54.2), turned to 180 degrees
- moved C14 63.8 mm to (162.0, 64.5), turned to 90 degrees
- moved C8 63.2 mm to (165.2, 54.2), turned to 90 degrees
- moved C11 62.7 mm to (163.5, 54.2), turned to 90 degrees
- moved C9 60.4 mm to (168.4, 79.2), turned to 180 degrees
- moved R12 59.8 mm to (170.0, 68.2), turned to 180 degrees
- moved R6 57.9 mm to (154.8, 79.5), turned to -90 degrees
- moved C10 57.8 mm to (174.8, 59.2), turned to 0 degrees
- moved U3 54.9 mm to (168.0, 62.0), turned to -90 degrees
- moved J1 54.1 mm to (153.0, 85.8), turned to 0 degrees
- moved C12 52.3 mm to (173.2, 66.5)
- moved C13 52.3 mm to (173.2, 68.0)
- moved R3 50.5 mm to (161.2, 58.8)
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Connections:
- C1 pad 1: VBUS -> /VUSB
- C15 pad 1: /VBAT -> +BATT
- J1 pad A4: VBUS -> /VUSB
- J1 pad A9: VBUS -> /VUSB
- J1 pad B4: VBUS -> /VUSB
- J1 pad B9: VBUS -> /VUSB
- J3 pad 1: unconnected-(J3-Pin_1-Pad1) -> +3V3
- J3 pad 2: unconnected-(J3-Pin_2-Pad2) -> GND
- J3 pad 3: unconnected-(J3-Pin_3-Pad3) -> /DCF77_OUT
- J3 pad 4: unconnected-(J3-Pin_4-Pad4) -> /DCF77_PON
- L1 pad 1: /VBAT -> +BATT
- Q1 pad 1: +5V -> VBUS
- Q1 pad 2: VBUS -> +5VD
- Q1 pad 3: +5VD -> +5V
- Q2 pad 1: /Screen/RESET -> /Screen/GDR
- Q2 pad 2: /Screen/GDR -> Net-(D5-A)
- Q2 pad 3: Net-(D5-A) -> /Screen/RESET
- R11 pad 1: /VBAT -> VBUS
- R11 pad 2: +BATT -> /VUSB
- U1 pad 1: STATUS_BAT -> /STAT_BAT
- U1 pad 4: VBUS -> /VUSB
- U3 pad 12: unconnected-(U3-PA2-Pad12) -> /USR_LED
- U3 pad 19: unconnected-(U3-PB1-Pad19) -> /DCF77_PON
- U3 pad 29: unconnected-(U3-PA8-Pad29) -> /STAT_BAT
- U3 pad 46: unconnected-(U3-PB9-Pad46) -> /SCREEN_ONOFF
- U6 pad 1: +BATT -> /VUSB
- U6 pad 2: /VBAT -> VBUS
Routing:
- net /USB-: track 0.00 -> 2.41 mm
- net /USB+: track 0.00 -> 2.39 mm
- net Net-(J1-CC2): track 0.00 -> 1.74 mm
- net Net-(J1-CC1): track 0.00 -> 1.74 mm

Commit message: routing
Parts:
- added R20: 33, Resistor_SMD:R_0603_1608Metric, F.Cu at (178.0, 60.2)
- added R21: 33, Resistor_SMD:R_0603_1608Metric, F.Cu at (178.0, 61.8)
- added R22: 33, Resistor_SMD:R_0603_1608Metric, F.Cu at (178.0, 63.2)
- added TP1: SCL_INA219, TestPoint:TestPoint_Pad_D1.0mm, F.Cu at (165.5, 68.8)
- added TP2: SDA_INA219, TestPoint:TestPoint_Pad_D1.0mm, F.Cu at (167.0, 68.8)
- added TP3: VBAT_SENSE, TestPoint:TestPoint_Pad_D1.0mm, F.Cu at (118.4, 67.1)
- added TP4: DCF77_OUT, TestPoint:TestPoint_Pad_D1.0mm, F.Cu at (160.5, 61.7)
- added TP5: SPI_CLK, TestPoint:TestPoint_Pad_D1.0mm, F.Cu at (191.8, 57.9)
- added TP6: SPI_CS, TestPoint:TestPoint_Pad_D1.0mm, F.Cu at (191.8, 56.7)
- added TP7: SPI_DATA, TestPoint:TestPoint_Pad_D1.0mm, F.Cu at (191.8, 59.2)
- R13: value 330 -> 1k
- moved J1 55.9 mm to (103.8, 59.2), turned to -90 degrees
- moved R6 48.4 mm to (110.0, 61.0), turned to 180 degrees
- moved R7 47.0 mm to (110.0, 58.0), turned to 180 degrees
- moved R10 13.4 mm to (176.6, 67.2)
- moved D3 12.4 mm to (135.6, 65.8), turned to 180 degrees
- moved C18 11.9 mm to (181.4, 70.7)
- moved C17 11.7 mm to (135.1, 68.3), turned to -90 degrees
- moved C20 11.6 mm to (121.8, 64.3)
- moved C22 11.6 mm to (123.3, 64.3)
- moved R18 11.6 mm to (115.3, 64.3)
- moved R19 11.6 mm to (116.8, 64.3)
- moved U7 11.6 mm to (119.4, 63.8)
- moved U5 11.4 mm to (177.9, 70.7)
- moved C15 8.87 mm to (137.4, 71.5), turned to 90 degrees
- moved R5 8.68 mm to (179.2, 67.2)
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Connections:
- net Net-(D4-A) renamed /SW
- J2 pad 10: /SCREEN_RST_N -> /Screen/RST_N
- J2 pad 11: /SCREEN_DC -> /Screen/DC
- J2 pad 9: /SCREEN_BUSY_N -> /Screen/BUSY_N
Routing:
- net /SPI_CS: track 0.00 -> 40.4 mm, vias 0 -> 2
- net /SPI_CLK: track 0.00 -> 27.0 mm, vias 0 -> 2
- net /SPI_DATA: track 0.00 -> 25.4 mm, vias 0 -> 2
- net /Screen/RST_N: track 0.00 -> 20.7 mm
- net Net-(D5-A): track 0.00 -> 20.5 mm, vias 0 -> 2
- net /Screen/DC: track 0.00 -> 20.0 mm, vias 0 -> 2
- net /Screen/BUSY_N: track 0.00 -> 19.7 mm
- net +3V3: track 0.00 -> 16.6 mm
- net Net-(D5-K): track 0.00 -> 15.4 mm, vias 0 -> 2
- net /SCL_HDC1080: track 0.00 -> 11.8 mm
- net /DCF77_OUT: track 0.00 -> 10.1 mm
- net VBUS: track 0.00 -> 9.95 mm
- net /Screen/VCC: track 0.00 -> 9.16 mm
- net /SDA_HDC1080: track 0.00 -> 9.02 mm
- net +BATT: track 0.00 -> 8.32 mm
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- added copper zone on F.Cu, net +3V3
- added copper zone on F.Cu, net +5V
- added copper zone on F.Cu, net +5VD
- added copper zone on F.Cu, net +BATT
- added copper zone on F.Cu, net /SW
- added copper zone on F.Cu, net /VUSB
- added copper zone on F.Cu, net VBUS

Commit message: tbd diff pair config
Routing:
- net /USB+: track 2.39 -> 80.7 mm
- net /USB-: track 2.41 -> 80.3 mm
Other:
- copper layers 2 -> 4
- rule solder_mask_min_width: 0.12 -> 0.02
Changed lines of the file:
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@@
 (kicad_pcb (version 20221018) (generator pcbnew)
   (general
-    (thickness 1.6)
+    (thickness 1.60252)
   )
   (paper "A4")
   (layers
     (0 "F.Cu" signal "Front")
+    (1 "In1.Cu" signal)
+    (2 "In2.Cu" signal)
     (31 "B.Cu" signal "Back")
     (34 "B.Paste" user)
@@
       (layer "F.SilkS" (type "Top Silk Screen"))
       (layer "F.Paste" (type "Top Solder Paste"))
-      (layer "F.Mask" (type "Top Solder Mask") (thickness 0.01))
-      (layer "F.Cu" (type "copper") (thickness 0.035))
-      (layer "dielectric 1" (type "core") (thickness 1.51) (material "FR4") (epsilon_r 4.5) (loss_tangent 0.02))
-      (layer "B.Cu" (type "copper") (thickness 0.035))
-      (layer "B.Mask" (type "Bottom Solder Mask") (thickness 0.01))
+      (layer "F.Mask" (type "Top Solder Mask") (thickness 0.025))
+      (layer "F.Cu" (type "copper") (thickness 0.04))
+      (layer "dielectric 1" (type "core") (thickness 0.13626) (material "FR4") (epsilon_r 4.5) (loss_tangent 0.02))
+      (layer "In1.Cu" (type "copper") (thickness 0.035))
+      (layer "dielectric 2" (type "prepreg") (thickness 1.13) (material "FR4") (epsilon_r 4.5) (loss_tangent 0.02))
+      (layer "In2.Cu" (type "copper") (thickness 0.035))
+      (layer "dielectric 3" (type "core") (thickness 0.13626) (material "FR4") (epsilon_r 4.5) (loss_tangent 0.02))
+      (layer "B.Cu" (type "copper") (thickness 0.04))
+      (layer "B.Mask" (type "Bottom Solder Mask") (thickness 0.025))
       (layer "B.Paste" (type "Bottom Solder Paste"))
       (layer "B.SilkS" (type "Bottom Silk Screen"))
@@
     )
     (pad_to_mask_clearance 0)
-    (solder_mask_min_width 0.12)
+    (solder_mask_min_width 0.02)
     (pcbplotparams
       (layerselection 0x00010fc_ffffffff)
@@
     (fp_line (start 38.53 -10.33) (end 38.53 10.33)
       (stroke (width 0.1) (type solid)) (layer "F.Fab"))
-    (pad "" np_thru_hole circle (at -35.85 8) (size 2.4 2.4) (drill 3.45) (layers "F&B.Cu" "*.Mask"))
+    (pad "" np_thru_hole circle (at -35.85 8) (size 2.4 2.4) (drill 3.45) (layers "*.Cu" "*.Mask"))
     (pad "1" smd rect (at -39.33 0) (size 7.77 7.35) (layers "F.Cu" "F.Paste" "F.Mask")
       (net 2 "+BATT") (pinfunction "+") (pintype "passive"))
@@
     (fp_rect (start -4.47 -3.675) (end 4.47 3.675)
       (stroke (width 0.1) (type solid)) (fill none) (layer "F.Fab"))
-    (pad "" np_thru_hole circle (at -2.89 -2.605 270) (size 0.65 0.65) (drill 0.65) (layers "F&B.Cu" "*.Mask"))
-    (pad "" np_thru_hole circle (at 2.89 -2.605 270) (size 0.65 0.65) (drill 0.65) (layers "F&B.Cu" "*.Mask"))
+    (pad "" np_thru_hole circle (at -2.89 -2.605 270) (size 0.65 0.65) (drill 0.65) (layers "*.Cu" "*.Mask"))
+    (pad "" np_thru_hole circle (at 2.89 -2.605 270) (size 0.65 0.65) (drill 0.65) (layers "*.Cu" "*.Mask"))
     (pad "A1" smd rect (at -3.2 -3.68 270) (size 0.6 1.15) (layers "F.Cu" "F.Paste" "F.Mask")
       (net 1 "GND") (pinfunction "GND") (pintype "passive"))
@@
   (segment (start 136.3875 65.8) (end 137.7375 65.8) (width 0.127) (layer "F.Cu") (net 22))
   (segment (start 107.43 58) (end 109.175 58) (width 0.127) (layer "F.Cu") (net 23))
-  (segment (start 108.075 60) (end 107.43 60) (width 0.1524) (layer "F.Cu") (net 24))
-  (segment (start 108.2 59.125) (end 108.2 59.875) (width 0.1524) (layer "F.Cu") (net 24))
-  (segment (start 108.075 59) (end 108.2 59.125) (width 0.1524) (layer "F.Cu") (net 24))
+  (segment (start 108.634264 58.9087) (end 109.324264 59.5987) (width 0.1524) (layer "F.Cu") (net 24))
   (segment (start 108.2 59.875) (end 108.075 60) (width 0.1524) (layer "F.Cu") (net 24))
-  (segment (start 107.43 59) (end 108.075 59) (width 0.1524) (layer "F.Cu") (net 24))
+  (segment (start 169.1587 66.2538) (end 169.25 66.1625) (width 0.1524) (layer "F.Cu") (net 24))
+  (segment (start 107.43 59) (end 108.2 59) (width 0.1524) (layer "F.Cu") (net 24))
+  (segment (start 107.43 59) (end 107.4768 58.9532) (width 0.1524) (layer "F.Cu") (net 24))
+  (segment (start 108.075 60) (end 107.43 60) (width 0.1524) (layer "F.Cu") (net 24))
+  (segment (start 107.43 59) (end 108.292501 59) (width 0.1524) (layer "F.Cu") (net 24))
+  (segment (start 109.324264 59.5987) (end 111.404264 59.5987) (width 0.1524) (layer "F.Cu") (net 24))
+  (segment (start 108.383801 58.9087) (end 108.634264 58.9087) (width 0.1524) (layer "F.Cu") (net 24))
+  (segment (start 120.114264 74.3987) (end 165.995736 74.3987) (width 0.1524) (layer "F.Cu") (net 24))
+  (segment (start 111.404264 59.5987) (end 112.0613 60.255736) (width 0.1524) (layer "F.Cu") (net 24))
+  (segment (start 108.2 59) (end 108.2 59.875) (width 0.1524) (layer "F.Cu") (net 24))
+  (segment (start 165.995736 74.3987) (end 169.1587 71.235736) (width 0.1524) (layer "F.Cu") (net 24))
+  (segment (start 108.292501 59) (end 108.383801 58.9087) (width 0.1524) (layer "F.Cu") (net 24))
+  (segment (start 112.0613 60.255736) (end 112.0613 66.345736) (width 0.1524) (layer "F.Cu") (net 24))
+  (segment (start 112.0613 66.345736) (end 120.114264 74.3987) (width 0.1524) (layer "F.Cu") (net 24))
+  (segment (start 107.4768 58.9532) (end 107.5 58.9532) (width 0.1524) (layer "F.Cu") (net 24))
+  (segment (start 169.1587 71.235736) (end 169.1587 66.2538) (width 0.1524) (layer "F.Cu") (net 24))
+  (segment (start 107.43 58.5) (end 107.4768 58.5468) (width 0.1524) (layer "F.Cu") (net 25))
+  (segment (start 111.535736 59.2813) (end 112.3787 60.124264) (width 0.1524) (layer "F.Cu") (net 25))
+  (segment (start 112.3787 60.124264) (end 112.3787 66.214264) (width 0.1524) (layer "F.Cu") (net 25))
+  (segment (start 168.8413 68.909185) (end 168.6088 68.676685) (width 0.1524) (layer "F.Cu") (net 25))
+  (segment (start 107.4768 58.5468) (end 107.5 58.5468) (width 0.1524) (layer "F.Cu") (net 25))
+  (segment (start 107.43 58.5) (end 108.292501 58.5) (width 0.1524) (layer "F.Cu") (net 25))
+  (segment (start 168.8413 67.590815) (end 168.8413 66.2538) (width 0.1524) (layer "F.Cu") (net 25))
+  (segment (start 168.8413 66.2538) (end 168.75 66.1625) (width 0.1524) (layer "F.Cu") (net 25))
+  (segment (start 108.765736 58.5913) (end 109.455736 59.2813) (width 0.1524) (layer "F.Cu") (net 25))
+  (segment (start 108.383801 58.5913) (end 108.765736 58.5913) (width 0.1524) (layer "F.Cu") (net 25))
   (segment (start 107.43 58.5) (end 106.75 58.5) (width 0.1524) (layer "F.Cu") (net 25))
+  (segment (start 165.864264 74.0813) (end 168.8413 71.104264) (width 0.1524) (layer "F.Cu") (net 25))
   (segment (start 106.75 59.5) (end 107.43 59.5) (width 0.1524) (layer "F.Cu") (net 25))
+  (segment (start 168.8413 71.104264) (end 168.8413 68.909185) (width 0.1524) (layer "F.Cu") (net 25))
+  (segment (start 109.455736 59.2813) (end 111.535736 59.2813) (width 0.1524) (layer "F.Cu") (net 25))
+  (segment (start 112.3787 66.214264) (end 120.245736 74.0813) (width 0.1524) (layer "F.Cu") (net 25))
   (segment (start 106.75 58.5) (end 106.6888 58.5612) (width 0.1524) (layer "F.Cu") (net 25))
+  (segment (start 168.6088 68.676685) (end 168.6088 67.823315) (width 0.1524) (layer "F.Cu") (net 25))
   (segment (start 106.6888 59.4388) (end 106.75 59.5) (width 0.1524) (layer "F.Cu") (net 25))
+  (segment (start 168.6088 67.823315) (end 168.8413 67.590815) (width 0.1524) (layer "F.Cu") (net 25))
   (segment (start 106.6888 58.5612) (end 106.6888 59.4388) (width 0.1524) (layer "F.Cu") (net 25))
+  (segment (start 108.292501 58.5) (end 108.383801 58.5913) (width 0.1524) (layer "F.Cu") (net 25))
+  (segment (start 120.245736 74.0813) (end 165.864264 74.0813) (width 0.1524) (layer "F.Cu") (net 25))
   (segment (start 107.43 61) (end 109.175 61) (width 0.127) (layer "F.Cu") (net 28))
   (segment (start 192.6 52.975) (end 192.575 53) (width 0.25) (layer "F.Cu") (net 29))
@@
       00000000-0000-0000-0000-00006116cca6
       00000000-0000-0000-0000-000061919138
-      15c4342e-9310-4cf4-b483-95f3f5840c2f
       25624e47-e3c8-40f4-97f5-a110260862b0
       99df4698-dac4-4260-912b-5ca550f8804f
       a12b57d1-dc57-45ff-90e9-1def28254f06
-      a257361d-190e-4fb6-9a7f-a1358d76336c
-      a2bfc09c-a5af-43b8-a77a-0ba2dd009aaa
       b547ba26-f86e-479d-9c7c-3f9f3a913ef0
-      cb41d96a-e287-4155-8864-d13db31485e2
       d875407b-a93d-4917-abdb-227229639ce5
-      e37f3687-52f6-413b-92bd-100cb672df75
       e6a02919-5c8f-4346-b180-f03dd590a500
       ed99435d-4b45-4988-80b9-f6d46e13d36d

Commit message: maj
Parts:
- removed C19: 100n, Capacitor_SMD:C_0603_1608Metric
- removed R11: 300m, Resistor_SMD:R_0805_2012Metric
- removed R14, R15: 4k7, Resistor_SMD:R_0603_1608Metric
- removed R16, R17: 0, Resistor_SMD:R_0603_1608Metric
- removed TP1: SCL_INA219, TestPoint:TestPoint_Pad_D1.0mm
- removed TP2: SDA_INA219, TestPoint:TestPoint_Pad_D1.0mm
- removed U6: INA219AxDCN, Package_TO_SOT_SMD:SOT-23-8
- moved R12 1.29 mm to (170.3, 69.5)
Connections:
- C1 pad 1: /VUSB -> VBUS
- J1 pad A4: /VUSB -> VBUS
- J1 pad A9: /VUSB -> VBUS
- J1 pad B4: /VUSB -> VBUS
- J1 pad B9: /VUSB -> VBUS
- U1 pad 4: /VUSB -> VBUS
Routing:
- net GND: track 8.22 -> 29.2 mm, vias 5 -> 22
- net /SCREEN_ONOFF: track 0.00 -> 14.4 mm
- net +3V3: track 16.6 -> 30.1 mm, vias 0 -> 16
- net Net-(U3-PF0): track 0.00 -> 7.85 mm
- net VBUS: track 9.95 -> 2.47 mm, vias 0 -> 7
- net /Screen/VCC: track 9.16 -> 15.9 mm, vias 0 -> 2
- net /VUSB: track 6.33 -> 0.00 mm
- net /SCL_INA219: track 6.09 -> 0.00 mm
- net /USB+: track 80.7 -> 86.7 mm
- net Net-(U3-PF1): track 0.00 -> 5.60 mm
- net /SDA_INA219: track 5.49 -> 0.00 mm
- net /USB-: track 80.3 -> 85.8 mm
- net Net-(U6-A0): track 5.46 -> 0.00 mm
- net Net-(Q3-G): track 0.00 -> 1.66 mm
- net Net-(U6-A1): track 1.60 -> 0.00 mm
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- added copper zone on In2.Cu, net +3V3
- added copper zone on In2.Cu, net +BATT
- added copper zone on In1.Cu, net GND
- added copper zone on In2.Cu, net VBUS
- removed copper zone on F.Cu, net /VUSB
