File: DCF77_Horloge.kicad_pcb (KiCad board)
At the start: 4 copper layers, 98.6 x 61.3 mm, 80 parts, among them J1 USB_C_Receptacle_USB2.0, J2 FH34SRJ 24S, J3 Conn_01x04_Socket, Q1 AO3401A, Q2 SK3424, Q3 SK3424, SW1 BOOT, SW3 RST, U1 MCP73831-2-OT, U2 NCP1117-3.3_SOT223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

Commit message: board to fab
Routing:
- net /VBAT_SENSE: track 4.00 -> 72.2 mm
- net /STAT_BAT: track 0.00 -> 49.7 mm, vias 0 -> 2
- net /BOOT0: track 0.00 -> 29.3 mm
- net /RST: track 0.00 -> 27.5 mm, vias 0 -> 2
- net +5V: track 3.04 -> 24.4 mm
- net +3V3: track 30.1 -> 40.8 mm, vias 16 -> 23
- net GND: track 29.2 -> 37.8 mm, vias 22 -> 80
- net Net-(U1-PROG): track 0.00 -> 1.73 mm
- net unconnected-(U5-DAP-Pad7): vias 0 -> 6
- added copper zone on B.Cu, net GND
- added copper zone on F.Cu, net GND
- added copper zone on In2.Cu, net GND
- added copper zone on In1.Cu, net unconnected-(U5-DAP-Pad7)
Other:
- board text added: "3V3"
- board text added: "BOOT"
- board text added: "CS CLK DATA"
- board text added: "DCF77_Clock Rev1"
- board text added: "OUT"
- board text added: "PON"
- board text added: "RESET"
- board text added: "VBAT"
- board text removed: "3.3V"
- board text removed: "SCL"
- board text removed: "SDA"
