File: DCF77_Horloge.kicad_sch (KiCad schematic)
At the start: 60 parts, among them J1 USB_C_Receptacle_USB2.0, J3 Conn_01x04_Socket, Q1 AO3401A, SW1 BOOT, SW3 RST, U1 MCP73831-2-OT, U2 NCP1117-3.3_SOT223, U3 STM32F302C6Tx, U4 TPS613222ADBV, U5 HDC1080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

Commit message: update pdf
Connections:
- net USR_LED: now also U3.12 (PA2)
Other:
- moved on the sheet: D2, R3
Changed lines of the file:
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@@
     (stroke (width 0) (type default))
   )
+  (wire (pts (xy 101.6 142.24) (xy 92.71 142.24))
+    (stroke (width 0) (type default))
+  )
   (wire (pts (xy 266.7 92.71) (xy 280.67 92.71))
     (stroke (width 0) (type default))
@@
     (stroke (width 0) (type default))
   )
-  (wire (pts (xy 33.02 187.96) (xy 27.94 187.96))
+  (wire (pts (xy 36.83 171.45) (xy 41.91 171.45))
     (stroke (width 0) (type default))
   )
@@
     (stroke (width 0) (type default))
   )
-  (wire (pts (xy 20.32 187.96) (xy 17.78 187.96))
+  (wire (pts (xy 49.53 171.45) (xy 52.07 171.45))
     (stroke (width 0) (type default))
   )
@@
     (stroke (width 0) (type default))
   )
+  (wire (pts (xy 20.32 171.45) (xy 29.21 171.45))
+    (stroke (width 0) (type default))
+  )
   (wire (pts (xy 248.92 82.55) (xy 248.92 83.82))
     (stroke (width 0) (type default))
@@
     (stroke (width 0) (type default))
   )
-  (wire (pts (xy 40.64 187.96) (xy 54.61 187.96))
-    (stroke (width 0) (type default))
-  )
   (wire (pts (xy 156.21 48.26) (xy 161.29 48.26))
     (stroke (width 0) (type default))
@@
     (effects (font (size 1.27 1.27)) (justify left bottom))
   )
-  (label "USR_LED" (at 43.18 187.96 0) (fields_autoplaced)
+  (label "USR_LED" (at 20.32 171.45 0) (fields_autoplaced)
     (effects (font (size 1.27 1.27)) (justify left bottom))
   )
@@
     (effects (font (size 1.27 1.27)) (justify left bottom))
   )
+  (label "USR_LED" (at 101.6 142.24 180) (fields_autoplaced)
+    (effects (font (size 1.27 1.27)) (justify right bottom))
+  )
   (label "SCREEN_BUSY_N" (at 120.65 137.16 0) (fields_autoplaced)
     (effects (font (size 1.27 1.27)) (justify left bottom))
@@
     )
   )
-  (symbol (lib_id "Device:R") (at 24.13 187.96 90) (unit 1)
+  (symbol (lib_id "Device:R") (at 45.72 171.45 270) (unit 1)
     (in_bom yes) (on_board yes) (dnp no)
-    (property "Reference" "R3" (at 24.13 190.5 90)
+    (property "Reference" "R3" (at 45.72 168.91 90)
       (effects (font (size 1.27 1.27)))
     )
-    (property "Value" "270" (at 24.13 187.96 90)
+    (property "Value" "270" (at 45.72 171.45 90)
       (effects (font (size 1.27 1.27)))
     )
-    (property "Footprint" "Resistor_SMD:R_0603_1608Metric" (at 24.13 189.738 90)
+    (property "Footprint" "Resistor_SMD:R_0603_1608Metric" (at 45.72 169.672 90)
       (effects (font (size 1.27 1.27)) hide)
     )
-    (property "Datasheet" "~" (at 24.13 187.96 0)
+    (property "Datasheet" "~" (at 45.72 171.45 0)
       (effects (font (size 1.27 1.27)) hide)
     )
@@
     )
   )
-  (symbol (lib_id "power:GND") (at 17.78 187.96 0) (unit 1)
+  (symbol (lib_id "power:GND") (at 52.07 171.45 0) (unit 1)
     (in_bom yes) (on_board yes) (dnp no)
-    (property "Reference" "#PWR014" (at 17.78 194.31 0)
+    (property "Reference" "#PWR014" (at 52.07 177.8 0)
       (effects (font (size 1.27 1.27)) hide)
     )
-    (property "Value" "GND" (at 17.907 192.3542 0)
+    (property "Value" "GND" (at 52.197 175.8442 0)
       (effects (font (size 1.27 1.27)))
     )
-    (property "Footprint" "" (at 17.78 187.96 0)
+    (property "Footprint" "" (at 52.07 171.45 0)
       (effects (font (size 1.27 1.27)) hide)
     )
-    (property "Datasheet" "" (at 17.78 187.96 0)
+    (property "Datasheet" "" (at 52.07 171.45 0)
       (effects (font (size 1.27 1.27)) hide)
     )
@@
     )
   )
-  (symbol (lib_id "Device:LED") (at 36.83 187.96 0) (unit 1)
+  (symbol (lib_id "Device:LED") (at 33.02 171.45 180) (unit 1)
     (in_bom yes) (on_board yes) (dnp no)
-    (property "Reference" "D2" (at 40.64 186.69 0)
+    (property "Reference" "D2" (at 29.21 172.72 0)
       (effects (font (size 1.27 1.27)) (justify right))
     )
-    (property "Value" "LED_DEBUG" (at 38.1 191.77 0)
+    (property "Value" "LED_DEBUG" (at 31.75 167.64 0)
       (effects (font (size 1.27 1.27)) (justify right))
     )
-    (property "Footprint" "LED_SMD:LED_0603_1608Metric" (at 36.83 187.96 0)
+    (property "Footprint" "LED_SMD:LED_0603_1608Metric" (at 33.02 171.45 0)
       (effects (font (size 1.27 1.27)) hide)
     )
-    (property "Datasheet" "~" (at 36.83 187.96 0)
+    (property "Datasheet" "~" (at 33.02 171.45 0)
       (effects (font (size 1.27 1.27)) hide)
     )

Commit message: update
Parts:
- added Q2: SK3424, Package_TO_SOT_SMD:SC-59, symbol Device:Q_NMOS_GSD
- added R9: 120, Resistor_SMD:R_0603_1608Metric, symbol Device:R
- BT1: footprint Battery:BatteryHolder_MPD_BH-18650-PC2 -> Battery:BatteryHolder_Keystone_1042_1x18650
- J1: footprint Connector_USB:USB_C_Receptacle_GCT_USB4085 -> Connector_USB:USB_C_Receptacle_GCT_USB4105-xx-A_16P_TopMnt_Horizontal
- J3: footprint Connector_PinHeader_2.54mm:PinHeader_1x04_P2.54mm_Vertical -> Connector_PinHeader_2.54mm:PinHeader_1x04_P2.54mm_Vertical_SMD_Pin1Left
- Q1: symbol Device:Q_PMOS_DGS -> Device:Q_PMOS_GSD
- R11: footprint Resistor_SMD:R_2512_6332Metric -> Resistor_SMD:R_0805_2012Metric
Connections:
- net STATUS_BAT is gone; now on net STAT_BAT: U1.1 (STAT)
- net +3V3: now also J3.1 (Pin_1), Q2.3 (D)
- net +5V: now also Q1.3 (D); no longer Q1.1 (D)
- net +5VD: now also Q1.2 (S); no longer Q1.3 (S)
- net +BATT: now also C15.1, L1.1; no longer R11.2, U6.1 (IN+)
- net DCF77_OUT: now also J3.3 (Pin_3)
- net GND: now also J3.2 (Pin_2)
- net Screen/VCC: now also Q2.2 (S)
- net VBUS: now also Q1.1 (G), R11.1, U6.2 (IN-); no longer C1.1, J1.A4 (VBUS), J1.A9 (VBUS), J1.B4 (VBUS), J1.B9 (VBUS), Q1.2 (G), U1.4 (VDD)
- net DCF77_PON: now reaches J3.4 (Pin_4)
- net DCF77_PON: now also U3.19 (PB1)
- net STAT_BAT: now reaches U3.29 (PA8)
- net SCREEN_ONOFF: now reaches U3.46 (PB9)
- net SCREEN_ONOFF: now also R9.1
- removed net VBAT: C15.1, L1.1, R11.1, U6.2 (IN-)
- new net: Q2.1 (G), R9.2
- new net VUSB: C1.1, J1.A4 (VBUS), J1.A9 (VBUS), J1.B4 (VBUS), J1.B9 (VBUS), R11.2, U1.4 (VDD), U6.1 (IN+)
Other:
- note added: "PON active Low"
- moved on the sheet: C3, J3, R11

Commit message: routing
Parts:
- added R20, R21, R22: 33, Resistor_SMD:R_0603_1608Metric, symbol Device:R
- added TP1: SCL_INA219, TestPoint:TestPoint_Pad_D1.0mm, symbol Connector:TestPoint
- added TP2: SDA_INA219, TestPoint:TestPoint_Pad_D1.0mm, symbol Connector:TestPoint
- added TP3: VBAT_SENSE, TestPoint:TestPoint_Pad_D1.0mm, symbol Connector:TestPoint
- added TP4: DCF77_OUT, TestPoint:TestPoint_Pad_D1.0mm, symbol Connector:TestPoint
- added TP5: SPI_CLK, TestPoint:TestPoint_Pad_D1.0mm, symbol Connector:TestPoint
- added TP6: SPI_CS, TestPoint:TestPoint_Pad_D1.0mm, symbol Connector:TestPoint
- added TP7: SPI_DATA, TestPoint:TestPoint_Pad_D1.0mm, symbol Connector:TestPoint
- R13: value 330 -> 1k
Connections:
- net DCF77_OUT: now also TP4.1
- net SCL_INA219: now also TP1.1
- net SCREEN_BUSY_N: now also R20.1
- net SCREEN_DC: now also R22.1
- net SCREEN_RST_N: now also R21.1
- net SDA_INA219: now also TP2.1
- net SPI_CLK: now also TP5.1
- net SPI_CS: now also TP6.1
- net SPI_DATA: now also TP7.1
- net VBAT_SENSE: now also TP3.1
- net SW: now reaches D4.2 (A), L1.2, U4.1 (SW)
- new net Screen/BUSY_N: R20.2
- new net Screen/DC: R22.2
- new net Screen/RST_N: R21.2

Commit message: maj
Parts:
- removed C19: 100n, Capacitor_SMD:C_0603_1608Metric, symbol Device:C
- removed R11: 300m, Resistor_SMD:R_0805_2012Metric, symbol Device:R
- removed R14, R15: 4k7, Resistor_SMD:R_0603_1608Metric, symbol Device:R
- removed R16, R17: 0, Resistor_SMD:R_0603_1608Metric, symbol Device:R
- removed TP1: SCL_INA219, TestPoint:TestPoint_Pad_D1.0mm, symbol Connector:TestPoint
- removed TP2: SDA_INA219, TestPoint:TestPoint_Pad_D1.0mm, symbol Connector:TestPoint
- removed U6: INA219AxDCN, Package_TO_SOT_SMD:SOT-23-8, symbol Sensor_Energy:INA219AxDCN
Connections:
- net VUSB is gone; now on net VBUS: C1.1, J1.A4 (VBUS), J1.A9 (VBUS), J1.B4 (VBUS), J1.B9 (VBUS), U1.4 (VDD)
Other:
- note removed: "Adress = 0b1000100 / 0x44"
- moved on the sheet: C20, C22, R18, R19, TP3, U7
